File: kicad_robot/kicad_robot_small.sch (KiCad schematic (older format))
At the start: 23 parts

Commit message: KiCAD
Parts:
- added U?: TSR_1-2433, Converter_DCDC:Converter_DCDC_TRACO_TSR-1_THT, symbol Regulator_Switching:TSR_1-2433
Connections:
- net +12V: now also U?.1 (Vin)
- net +3V3: now also U?.3 (Vout)
- net GND: now also U?.2 (GND)
- net 5V_Converti renamed +5V
Changed lines of the file:
@@
 	0    1    1    0
 $EndComp
-Wire Wire Line
-	4225 7650 5025 7650
-Text Label 5025 7650 2    50   ~ 0
-5V_Converti
 $Comp
 L Sensor_Current:ACS722xLCTR-05AB U?
@@
 	0    1    1    0
 $EndComp
+$Comp
+L Regulator_Switching:TSR_1-2433 U?
+U 1 1 6035A95D
+P 3825 8625
+F 0 "U?" H 3825 8992 50  0000 C CNN
+F 1 "TSR_1-2433" H 3825 8901 50  0000 C CNN
+F 2 "Converter_DCDC:Converter_DCDC_TRACO_TSR-1_THT" H 3825 8475 50  0001 L CIN
+F 3 "http://www.tracopower.com/products/tsr1.pdf" H 3825 8625 50  0001 C CNN
+	1    3825 8625
+	1    0    0    -1
+$EndComp
+$Comp
+L power:+5V #PWR?
+U 1 1 60360E0E
+P 4225 7650
+F 0 "#PWR?" H 4225 7500 50  0001 C CNN
+F 1 "+5V" V 4240 7778 50  0000 L CNN
+F 2 "" H 4225 7650 50  0001 C CNN
+F 3 "" H 4225 7650 50  0001 C CNN
+	1    4225 7650
+	0    1    1    0
+$EndComp
+$Comp
+L power:+12V #PWR?
+U 1 1 603616FA
+P 3425 8525
+F 0 "#PWR?" H 3425 8375 50  0001 C CNN
+F 1 "+12V" V 3440 8653 50  0000 L CNN
+F 2 "" H 3425 8525 50  0001 C CNN
+F 3 "" H 3425 8525 50  0001 C CNN
+	1    3425 8525
+	0    -1   -1   0
+$EndComp
+$Comp
+L power:GND #PWR?
+U 1 1 60362802
+P 3825 8825
+F 0 "#PWR?" H 3825 8575 50  0001 C CNN
+F 1 "GND" H 3830 8652 50  0000 C CNN
+F 2 "" H 3825 8825 50  0001 C CNN
+F 3 "" H 3825 8825 50  0001 C CNN
+	1    3825 8825
+	1    0    0    -1
+$EndComp
+$Comp
+L power:+3.3V #PWR?
+U 1 1 6036A6D3
+P 4225 8525
+F 0 "#PWR?" H 4225 8375 50  0001 C CNN
+F 1 "+3.3V" V 4240 8653 50  0000 L CNN
+F 2 "" H 4225 8525 50  0001 C CNN
+F 3 "" H 4225 8525 50  0001 C CNN
+	1    4225 8525
+	0    1    1    0
+$EndComp

Commit message: KiCad
Parts:
- removed U?: TSR_1-2433, Converter_DCDC:Converter_DCDC_TRACO_TSR-1_THT, symbol Regulator_Switching:TSR_1-2433
- added J? (x2): Conn_01x03_Female, symbol Connector:Conn_01x03_Female
Changed lines of the file:
@@
-$EndComp
-$Comp
-L Regulator_Switching:TSR_1-2433 U?
-U 1 1 6035A95D
-P 3825 8625
-F 0 "U?" H 3825 8992 50  0000 C CNN
-F 1 "TSR_1-2433" H 3825 8901 50  0000 C CNN
-F 2 "Converter_DCDC:Converter_DCDC_TRACO_TSR-1_THT" H 3825 8475 50  0001 L CIN
-F 3 "http://www.tracopower.com/products/tsr1.pdf" H 3825 8625 50  0001 C CNN
-	1    3825 8625
-	1    0    0    -1
 $EndComp
 $Comp
@@
 $EndComp
 $Comp
-L power:+12V #PWR?
-U 1 1 603616FA
-P 3425 8525
-F 0 "#PWR?" H 3425 8375 50  0001 C CNN
-F 1 "+12V" V 3440 8653 50  0000 L CNN
-F 2 "" H 3425 8525 50  0001 C CNN
-F 3 "" H 3425 8525 50  0001 C CNN
-	1    3425 8525
-	0    -1   -1   0
-$EndComp
-$Comp
-L power:GND #PWR?
-U 1 1 60362802
-P 3825 8825
-F 0 "#PWR?" H 3825 8575 50  0001 C CNN
-F 1 "GND" H 3830 8652 50  0000 C CNN
-F 2 "" H 3825 8825 50  0001 C CNN
-F 3 "" H 3825 8825 50  0001 C CNN
-	1    3825 8825
+L Connector:Conn_01x03_Female J?
+U 1 1 6031A117
+P 14275 1950
+F 0 "J?" H 14303 1976 50  0000 L CNN
+F 1 "Conn_01x03_Female" H 14303 1885 50  0000 L CNN
+F 2 "" H 14275 1950 50  0001 C CNN
+F 3 "~" H 14275 1950 50  0001 C CNN
+	1    14275 1950
 	1    0    0    -1
 $EndComp
 $Comp
-L power:+3.3V #PWR?
-U 1 1 6036A6D3
-P 4225 8525
-F 0 "#PWR?" H 4225 8375 50  0001 C CNN
-F 1 "+3.3V" V 4240 8653 50  0000 L CNN
-F 2 "" H 4225 8525 50  0001 C CNN
-F 3 "" H 4225 8525 50  0001 C CNN
-	1    4225 8525
-	0    1    1    0
+L Connector:Conn_01x03_Female J?
+U 1 1 6031D53E
+P 14275 2475
+F 0 "J?" H 14303 2501 50  0000 L CNN
+F 1 "Conn_01x03_Female" H 14303 2410 50  0000 L CNN
+F 2 "" H 14275 2475 50  0001 C CNN
+F 3 "~" H 14275 2475 50  0001 C CNN
+	1    14275 2475
+	1    0    0    -1
 $EndComp
 $EndSCHEMATC

Commit message: KiCAD
Parts:
- removed J?: Conn_01x03_Female, symbol Connector:Conn_01x03_Female
- added J? (x4): Conn_01x03_Female, symbol Connector:Conn_01x03_Female
- added R? (x5): 10k, symbol Device:R
Connections:
- net +5V: now also J?.1 (Pin_1), J?.1 (Pin_1), J?.1 (Pin_1), J?.1 (Pin_1), J?.1 (Pin_1)
- net GND: now also J?.3 (Pin_3), J?.3 (Pin_3), J?.3 (Pin_3), J?.3 (Pin_3), J?.3 (Pin_3), R?.2, R?.2, R?.2, R?.2, R?.2
- net POMPE_1: now also R?.1
- net POMPE_2: now also R?.1
- net POMPE_3: now also R?.1
- net POMPE_4: now also R?.1
- net POMPE_5: now also R?.1
- net SERVO_1: now also J?.2 (Pin_2)
- net SERVO_2: now also J?.2 (Pin_2)
- net SERVO_3: now also J?.2 (Pin_2)
- net SERVO_4: now also J?.2 (Pin_2)
- net SERVO_5: now also J?.2 (Pin_2)

Commit message: KiCAD
Parts:
- added Q?: IRLML0030, Package_TO_SOT_SMD:SOT-23, symbol Transistor_FET:IRLML0030
- added R?: 10k, symbol Device:R
Connections:
- net EV_1: now also Q?.1 (G), R?.1
- net GND: now also Q?.2 (S), R?.2
Changed lines of the file:
@@
 Wire Wire Line
 	10950 7250 10400 7250
+$Comp
+L Transistor_FET:IRLML0030 Q?
+U 1 1 6038953D
+P 14225 5025
+F 0 "Q?" V 14567 5025 50  0000 C CNN
+F 1 "IRLML0030" V 14476 5025 50  0000 C CNN
+F 2 "Package_TO_SOT_SMD:SOT-23" H 14425 4950 50  0001 L CIN
+F 3 "https://www.infineon.com/dgdl/irlml0030pbf.pdf?fileId=5546d462533600a401535664773825df" H 14225 5025 50  0001 L CNN
+	1    14225 5025
+	0    1    -1   0
+$EndComp
+Wire Wire Line
+	14225 5225 14225 5425
+Wire Wire Line
+	14225 5425 14000 5425
+Text Label 13550 5425 0    50   ~ 0
+EV_1
+$Comp
+L Device:R R?
+U 1 1 603A52E1
+P 14000 5575
+F 0 "R?" H 14070 5621 50  0000 L CNN
+F 1 "10k" H 14070 5530 50  0000 L CNN
+F 2 "" V 13930 5575 50  0001 C CNN
+F 3 "~" H 14000 5575 50  0001 C CNN
+	1    14000 5575
+	1    0    0    -1
+$EndComp
+Connection ~ 14000 5425
+Wire Wire Line
+	14000 5425 13550 5425
+$Comp
+L power:GND #PWR?
+U 1 1 603A64DA
+P 14000 5725
+F 0 "#PWR?" H 14000 5475 50  0001 C CNN
+F 1 "GND" H 14005 5552 50  0000 C CNN
+F 2 "" H 14000 5725 50  0001 C CNN
+F 3 "" H 14000 5725 50  0001 C CNN
+	1    14000 5725
+	1    0    0    -1
+$EndComp
+$Comp
+L power:GND #PWR?
+U 1 1 603A74C2
+P 14025 4925
+F 0 "#PWR?" H 14025 4675 50  0001 C CNN
+F 1 "GND" V 14030 4797 50  0000 R CNN
+F 2 "" H 14025 4925 50  0001 C CNN
+F 3 "" H 14025 4925 50  0001 C CNN
+	1    14025 4925
+	0    1    1    0
+$EndComp
+Wire Wire Line
+	14425 4925 15100 4925
 $EndSCHEMATC
