File: kicad_robot/kicad_robot_servos_ev_pompes.sch (KiCad schematic (older format))
At the start: 35 parts

Commit message: KICAD
Parts:
- removed C? (x4): 0.1µF, symbol Device:C
- removed C? (x4): 10nF, symbol Device:C
- removed J? (x4): Conn_01x03_Female, symbol Connector:Conn_01x03_Female
- removed Q? (x4): IRLML0030, Package_TO_SOT_SMD:SOT-23, symbol Transistor_FET:IRLML0030
- removed R? (x4): 10k, symbol Device:R
- removed U? (x4): ACS722xLCTR-05AB, Package_SO:SOIC-8_3.9x4.9mm_P1.27mm, symbol Sensor_Current:ACS722xLCTR-05AB
- added C? (x4): 0.1µF, symbol Device:C
- added C? (x4): 10nF, symbol Device:C
- added J?: Conn_SERVO_2, symbol Connector:Conn_01x03_Female
- added J?: Conn_SERVO_3, symbol Connector:Conn_01x03_Female
- added J?: Conn_SERVO_4, symbol Connector:Conn_01x03_Female
- added J?: Conn_SERVO_5, symbol Connector:Conn_01x03_Female
- added J?: Conn_POMPE_1, symbol Connector:Conn_01x02_Male
- added J?: Conn_POMPE_2, symbol Connector:Conn_01x02_Male
- added J?: Conn_POMPE_3, symbol Connector:Conn_01x02_Male
- added J?: Conn_POMPE_4, symbol Connector:Conn_01x02_Male
- added J?: Conn_POMPE_5, symbol Connector:Conn_01x02_Male
- added J?: Conn_EV_5, symbol Connector:Conn_01x02_Male
- added J?: Conn_EV_4, symbol Connector:Conn_01x02_Male
- added J?: Conn_EV_3, symbol Connector:Conn_01x02_Male
- added J?: Conn_EV_2, symbol Connector:Conn_01x02_Male
- added J?: Conn_EV_1, symbol Connector:Conn_01x02_Male
- added J?: Conn_I2C, symbol Connector:Conn_01x02_Male
- added J?: Screw_Terminal_POWER, symbol Connector:Screw_Terminal_01x02
- added Q? (x8): IRLML0030, Package_TO_SOT_SMD:SOT-23, symbol Transistor_FET:IRLML0030
- added R? (x8): 10k, symbol Device:R
- added R? (x4): R, symbol Device:R
- added U?: LM3940, Package_TO_SOT_SMD:SOT-223-3_TabPin2, symbol LM3940:LM3940
- added U? (x4): ACS722xLCTR-05AB, Package_SO:SOIC-8_3.9x4.9mm_P1.27mm, symbol Sensor_Current:ACS722xLCTR-05AB
- J?: value Conn_01x03_Female -> Conn_SERVO_1
Connections:
- net +12V: now also J?.2 (Pin_2), J?.2 (Pin_2), J?.2 (Pin_2), J?.2 (Pin_2), J?.2 (Pin_2), J?.2 (Pin_2), U?.1 (IP+), U?.1 (IP+), U?.1 (IP+), U?.1 (IP+), U?.2 (IP+), U?.2 (IP+), U?.2 (IP+), U?.2 (IP+)
- net +3V3: now also U?.2 (A1), U?.3 (A2), C?.2, C?.2, C?.2, C?.2, R?.1, R?.1, U?.3 (Vout), U?.8 (VCC), U?.8 (VCC), U?.8 (VCC), U?.8 (VCC)
- net +5V: now also J?.2 (Pin_2), J?.2 (Pin_2), J?.2 (Pin_2), J?.2 (Pin_2), J?.2 (Pin_2), U?.1 (Vin); no longer J?.1 (Pin_1)
- net ADC_2: now also C?.1, U?.7 (VIOUT)
- net ADC_3: now also C?.1, U?.7 (VIOUT)
- net ADC_4: now also C?.1, U?.7 (VIOUT)
- net ADC_5: now also C?.1, U?.7 (VIOUT)
- net EV_2: now also Q?.1 (G), R?.1
- net EV_3: now also Q?.1 (G), R?.1
- net EV_4: now also Q?.1 (G), R?.1
- net EV_5: now also Q?.1 (G), R?.1
- net EXT_SCL: now also J?.2 (Pin_2)
- net EXT_SDA: now also J?.1 (Pin_1)
- net GND: now also J?.1 (Pin_1), Q?.2 (S), U?.23 (~OE), U?.24 (A5), U?.25 (EXTCLK), U?.4 (A3), U?.5 (A4), U?.8 (A1), C?.1, C?.1, C?.1, C?.1, C?.2, C?.2, C?.2, C?.2, J?.1 (Pin_1), J?.1 (Pin_1), J?.1 (Pin_1), J?.1 (Pin_1), J?.1 (Pin_1), Q?.2 (S), Q?.2 (S), Q?.2 (S), Q?.2 (S), Q?.2 (S), Q?.2 (S), Q?.2 (S), Q?.2 (S), R?.1, R?.1, R?.2, R?.2, R?.2, R?.2, R?.2, R?.2, R?.2, R?.2, U?.2 (GND), U?.5 (GND), U?.5 (GND), U?.5 (GND), U?.5 (GND), U?.6 (BW_SEL), U?.6 (BW_SEL), U?.6 (BW_SEL), U?.6 (BW_SEL); no longer J?.3 (Pin_3)
- net POMPE_2: now also Q?.1 (G), R?.1
- net POMPE_3: now also Q?.1 (G), R?.1
- net POMPE_4: now also Q?.1 (G), R?.1
- net POMPE_5: now also Q?.1 (G), R?.1
- net SERVO_1: now also J?.3 (Pin_3); no longer J?.2 (Pin_2)
- net SERVO_2: now also J?.3 (Pin_3)
- net SERVO_3: now also J?.3 (Pin_3)
- net SERVO_4: now also J?.3 (Pin_3)
- net SERVO_5: now also J?.3 (Pin_3)
- net at U?.1 (A0): now also R?.2, R?.2
- net at U?.7 (A0): now also R?.2, R?.2
- net at U?.3 (IP-), U?.4 (IP-): now also J?.2 (Pin_2); no longer Q?.2 (S)
- net at Q?.3 (D): now also J?.1 (Pin_1)
- net 12V_POMPE_1: no longer names the net of Q?.3 (D)
- net 12V_POMPE_1: now also J?.1 (Pin_1)
- new net: J?.1 (Pin_1), Q?.3 (D) (x8)
- new net: J?.2 (Pin_2), U?.3 (IP-), U?.4 (IP-) (x4)
- no-connect marks 0 -> 6
Other:
- note added: "Ne souder que l'une\ndes deux résistances\n(Choix d'adresse)"
- moved on the sheet: C?, Q?, R?, U?

Commit message: KICAD
Parts:
- J? (x5): symbol Connector:Conn_01x03_Female -> Connector:Conn_01x03_Male
Connections:
- net GND: now also J?.3 (Pin_3), J?.3 (Pin_3), J?.3 (Pin_3), J?.3 (Pin_3), J?.3 (Pin_3); no longer J?.1 (Pin_1), J?.1 (Pin_1), J?.1 (Pin_1), J?.1 (Pin_1), J?.1 (Pin_1)
- net SERVO_1: now also J?.1 (Pin_1); no longer J?.3 (Pin_3)
- net SERVO_2: now also J?.1 (Pin_1); no longer J?.3 (Pin_3)
- net SERVO_3: now also J?.1 (Pin_1); no longer J?.3 (Pin_3)
- net SERVO_4: now also J?.1 (Pin_1); no longer J?.3 (Pin_3)
- net SERVO_5: now also J?.1 (Pin_1); no longer J?.3 (Pin_3)
Changed lines of the file:
@@
 $EndComp
 $Comp
-L Connector:Conn_01x03_Female J?
+L Connector:Conn_01x03_Male J?
 U 1 1 6031A117
-P 14275 1950
-F 0 "J?" H 14303 1976 50  0000 L CNN
-F 1 "Conn_SERVO_1" H 14303 1885 50  0000 L CNN
-F 2 "" H 14275 1950 50  0001 C CNN
-F 3 "~" H 14275 1950 50  0001 C CNN
-	1    14275 1950
-	1    0    0    -1
+P 14175 1925
+F 0 "J?" H 13612 1951 50  0000 L CNN
+F 1 "Conn_SERVO_1" H 13612 1860 50  0000 L CNN
+F 2 "" H 14175 1925 50  0001 C CNN
+F 3 "~" H 14175 1925 50  0001 C CNN
+	1    14175 1925
+	-1   0    0    1
 $EndComp
 $Comp
 L power:GND #PWR?
 U 1 1 603560D6
-P 14075 1850
-F 0 "#PWR?" H 14075 1600 50  0001 C CNN
-F 1 "GND" V 14080 1722 50  0000 R CNN
-F 2 "" H 14075 1850 50  0001 C CNN
-F 3 "" H 14075 1850 50  0001 C CNN
-	1    14075 1850
+P 13975 1825
+F 0 "#PWR?" H 13975 1575 50  0001 C CNN
+F 1 "GND" V 13980 1697 50  0000 R CNN
+F 2 "" H 13975 1825 50  0001 C CNN
+F 3 "" H 13975 1825 50  0001 C CNN
+	1    13975 1825
 	0    1    1    0
 $EndComp
@@
 L power:+5V #PWR?
 U 1 1 60356CC9
-P 14075 1950
-F 0 "#PWR?" H 14075 1800 50  0001 C CNN
-F 1 "+5V" V 14090 2078 50  0000 L CNN
-F 2 "" H 14075 1950 50  0001 C CNN
-F 3 "" H 14075 1950 50  0001 C CNN
-	1    14075 1950
-	0    -1   -1   0
-$EndComp
-Wire Wire Line
-	14075 2050 13325 2050
-Text Label 13325 2050 0    50   ~ 0
+P 13975 1925
+F 0 "#PWR?" H 13975 1775 50  0001 C CNN
+F 1 "+5V" V 13990 2053 50  0000 L CNN
+F 2 "" H 13975 1925 50  0001 C CNN
+F 3 "" H 13975 1925 50  0001 C CNN
+	1    13975 1925
+	0    -1   -1   0
+$EndComp
+Wire Wire Line
+	13975 2025 13225 2025
+Text Label 13225 2025 0    50   ~ 0
 SERVO_1
 $Comp
@@
 	14050 4100 14250 4100
 $Comp
-L Connector:Conn_01x03_Female J?
+L Connector:Conn_01x03_Male J?
 U 1 1 6035D969
-P 14275 2300
-F 0 "J?" H 14303 2326 50  0000 L CNN
-F 1 "Conn_SERVO_2" H 14303 2235 50  0000 L CNN
-F 2 "" H 14275 2300 50  0001 C CNN
-F 3 "~" H 14275 2300 50  0001 C CNN
-	1    14275 2300
-	1    0    0    -1
+P 14175 2275
+F 0 "J?" H 13612 2301 50  0000 L CNN
+F 1 "Conn_SERVO_2" H 13612 2210 50  0000 L CNN
+F 2 "" H 14175 2275 50  0001 C CNN
+F 3 "~" H 14175 2275 50  0001 C CNN
+	1    14175 2275
+	-1   0    0    1
 $EndComp
 $Comp
 L power:GND #PWR?
 U 1 1 6035D96F
-P 14075 2200
-F 0 "#PWR?" H 14075 1950 50  0001 C CNN
-F 1 "GND" V 14080 2072 50  0000 R CNN
-F 2 "" H 14075 2200 50  0001 C CNN
-F 3 "" H 14075 2200 50  0001 C CNN
-	1    14075 2200
+P 13975 2175
+F 0 "#PWR?" H 13975 1925 50  0001 C CNN
+F 1 "GND" V 13980 2047 50  0000 R CNN
+F 2 "" H 13975 2175 50  0001 C CNN
+F 3 "" H 13975 2175 50  0001 C CNN
+	1    13975 2175
 	0    1    1    0
 $EndComp
@@
 L power:+5V #PWR?
 U 1 1 6035D975
-P 14075 2300
-F 0 "#PWR?" H 14075 2150 50  0001 C CNN
-F 1 "+5V" V 14090 2428 50  0000 L CNN
-F 2 "" H 14075 2300 50  0001 C CNN
-F 3 "" H 14075 2300 50  0001 C CNN
-	1    14075 2300
-	0    -1   -1   0
-$EndComp
-Wire Wire Line
-	14075 2400 13325 2400
-Text Label 13325 2400 0    50   ~ 0
+P 13975 2275
+F 0 "#PWR?" H 13975 2125 50  0001 C CNN
+F 1 "+5V" V 13990 2403 50  0000 L CNN
+F 2 "" H 13975 2275 50  0001 C CNN
+F 3 "" H 13975 2275 50  0001 C CNN
+	1    13975 2275
+	0    -1   -1   0
+$EndComp
+Wire Wire Line
+	13975 2375 13225 2375
+Text Label 13225 2375 0    50   ~ 0
 SERVO_2
 $Comp
-L Connector:Conn_01x03_Female J?
+L Connector:Conn_01x03_Male J?
 U 1 1 60360D28
-P 14275 2650
-F 0 "J?" H 14303 2676 50  0000 L CNN
-F 1 "Conn_SERVO_3" H 14303 2585 50  0000 L CNN
-F 2 "" H 14275 2650 50  0001 C CNN
-F 3 "~" H 14275 2650 50  0001 C CNN
-	1    14275 2650
-	1    0    0    -1
+P 14175 2625
+F 0 "J?" H 13612 2651 50  0000 L CNN
+F 1 "Conn_SERVO_3" H 13612 2560 50  0000 L CNN
+F 2 "" H 14175 2625 50  0001 C CNN
+F 3 "~" H 14175 2625 50  0001 C CNN
+	1    14175 2625
+	-1   0    0    1
 $EndComp
 $Comp
 L power:GND #PWR?
 U 1 1 60360D2E
-P 14075 2550
-F 0 "#PWR?" H 14075 2300 50  0001 C CNN
-F 1 "GND" V 14080 2422 50  0000 R CNN
-F 2 "" H 14075 2550 50  0001 C CNN
-F 3 "" H 14075 2550 50  0001 C CNN
-	1    14075 2550
+P 13975 2525
+F 0 "#PWR?" H 13975 2275 50  0001 C CNN
+F 1 "GND" V 13980 2397 50  0000 R CNN
+F 2 "" H 13975 2525 50  0001 C CNN
+F 3 "" H 13975 2525 50  0001 C CNN
+	1    13975 2525
 	0    1    1    0
 $EndComp
@@
 L power:+5V #PWR?
 U 1 1 60360D34
-P 14075 2650
-F 0 "#PWR?" H 14075 2500 50  0001 C CNN
-F 1 "+5V" V 14090 2778 50  0000 L CNN
-F 2 "" H 14075 2650 50  0001 C CNN
-F 3 "" H 14075 2650 50  0001 C CNN
-	1    14075 2650
-	0    -1   -1   0
-$EndComp
-Wire Wire Line
-	14075 2750 13325 2750
-Text Label 13325 2750 0    50   ~ 0
+P 13975 2625
+F 0 "#PWR?" H 13975 2475 50  0001 C CNN
+F 1 "+5V" V 13990 2753 50  0000 L CNN
+F 2 "" H 13975 2625 50  0001 C CNN
+F 3 "" H 13975 2625 50  0001 C CNN
+	1    13975 2625
+	0    -1   -1   0
+$EndComp
+Wire Wire Line
+	13975 2725 13225 2725
+Text Label 13225 2725 0    50   ~ 0
 SERVO_3
 $Comp
-L Connector:Conn_01x03_Female J?
+L Connector:Conn_01x03_Male J?
 U 1 1 603641AD
-P 14275 3000
-F 0 "J?" H 14303 3026 50  0000 L CNN
-F 1 "Conn_SERVO_4" H 14303 2935 50  0000 L CNN
-F 2 "" H 14275 3000 50  0001 C CNN
-F 3 "~" H 14275 3000 50  0001 C CNN
-	1    14275 3000
-	1    0    0    -1
+P 14175 2975
+F 0 "J?" H 13612 3001 50  0000 L CNN
+F 1 "Conn_SERVO_4" H 13612 2910 50  0000 L CNN
+F 2 "" H 14175 2975 50  0001 C CNN
+F 3 "~" H 14175 2975 50  0001 C CNN
+	1    14175 2975
+	-1   0    0    1
 $EndComp
 $Comp
 L power:GND #PWR?
 U 1 1 603641B3
-P 14075 2900
-F 0 "#PWR?" H 14075 2650 50  0001 C CNN
-F 1 "GND" V 14080 2772 50  0000 R CNN
-F 2 "" H 14075 2900 50  0001 C CNN
-F 3 "" H 14075 2900 50  0001 C CNN
-	1    14075 2900
+P 13975 2875
+F 0 "#PWR?" H 13975 2625 50  0001 C CNN
+F 1 "GND" V 13980 2747 50  0000 R CNN
+F 2 "" H 13975 2875 50  0001 C CNN
+F 3 "" H 13975 2875 50  0001 C CNN
+	1    13975 2875
 	0    1    1    0
 $EndComp
@@
 L power:+5V #PWR?
 U 1 1 603641B9
-P 14075 3000
-F 0 "#PWR?" H 14075 2850 50  0001 C CNN
-F 1 "+5V" V 14090 3128 50  0000 L CNN
-F 2 "" H 14075 3000 50  0001 C CNN
-F 3 "" H 14075 3000 50  0001 C CNN
-	1    14075 3000
-	0    -1   -1   0
-$EndComp
-Wire Wire Line
-	14075 3100 13325 3100
-Text Label 13325 3100 0    50   ~ 0
+P 13975 2975
+F 0 "#PWR?" H 13975 2825 50  0001 C CNN
+F 1 "+5V" V 13990 3103 50  0000 L CNN
+F 2 "" H 13975 2975 50  0001 C CNN
+F 3 "" H 13975 2975 50  0001 C CNN
+	1    13975 2975
+	0    -1   -1   0
+$EndComp
+Wire Wire Line
+	13975 3075 13225 3075
+Text Label 13225 3075 0    50   ~ 0
 SERVO_4
 $Comp
-L Connector:Conn_01x03_Female J?
+L Connector:Conn_01x03_Male J?
 U 1 1 603675B3
-P 14275 3350
-F 0 "J?" H 14303 3376 50  0000 L CNN
-F 1 "Conn_SERVO_5" H 14303 3285 50  0000 L CNN
-F 2 "" H 14275 3350 50  0001 C CNN
-F 3 "~" H 14275 3350 50  0001 C CNN
-	1    14275 3350
-	1    0    0    -1
+P 14175 3325
+F 0 "J?" H 13612 3351 50  0000 L CNN
+F 1 "Conn_SERVO_5" H 13612 3260 50  0000 L CNN
+F 2 "" H 14175 3325 50  0001 C CNN
+F 3 "~" H 14175 3325 50  0001 C CNN
+	1    14175 3325
+	-1   0    0    1
 $EndComp
 $Comp
 L power:GND #PWR?
 U 1 1 603675B9
-P 14075 3250
-F 0 "#PWR?" H 14075 3000 50  0001 C CNN
-F 1 "GND" V 14080 3122 50  0000 R CNN
-F 2 "" H 14075 3250 50  0001 C CNN
-F 3 "" H 14075 3250 50  0001 C CNN
-	1    14075 3250
+P 13975 3225
+F 0 "#PWR?" H 13975 2975 50  0001 C CNN
+F 1 "GND" V 13980 3097 50  0000 R CNN
+F 2 "" H 13975 3225 50  0001 C CNN
+F 3 "" H 13975 3225 50  0001 C CNN
+	1    13975 3225
 	0    1    1    0
 $EndComp
@@
 L power:+5V #PWR?
 U 1 1 603675BF
-P 14075 3350
-F 0 "#PWR?" H 14075 3200 50  0001 C CNN
-F 1 "+5V" V 14090 3478 50  0000 L CNN
-F 2 "" H 14075 3350 50  0001 C CNN
-F 3 "" H 14075 3350 50  0001 C CNN
-	1    14075 3350
-	0    -1   -1   0
-$EndComp
-Wire Wire Line
-	14075 3450 13325 3450
-Text Label 13325 3450 0    50   ~ 0
+P 13975 3325
+F 0 "#PWR?" H 13975 3175 50  0001 C CNN
+F 1 "+5V" V 13990 3453 50  0000 L CNN
+F 2 "" H 13975 3325 50  0001 C CNN
+F 3 "" H 13975 3325 50  0001 C CNN
+	1    13975 3325
+	0    -1   -1   0
+$EndComp
+Wire Wire Line
+	13975 3425 13225 3425
+Text Label 13225 3425 0    50   ~ 0
 SERVO_5
 Wire Wire Line
