File: kicad_robot/kicad_robot_teensy.kicad_pcb (KiCad board)
At the start: 2 copper layers, 21 parts, among them Q1 IRLML0030, U12->5 R-78E5.0-1.0

Commit message: Routage de la carte Teensy V1.0
Parts:
- moved J_I2C->MULTIPLEX2 167.8 mm to (190.5, 95.2), turned to 180 degrees
- moved CONN->MD10_MOT_2 162.9 mm to (175.3, 128.3), turned to 270 degrees
- moved J_I2C->MULTIPLEX1 150.6 mm to (190.5, 82.5), turned to 180 degrees
- moved CONN->MD10_MOT_1 141.6 mm to (189.2, 128.3), turned to 270 degrees
- moved CONN->SERV_PAV1 124.1 mm to (189.2, 113.0)
- moved CARTE_MICR_COTROL1 123.3 mm to (152.4, 106.7), turned to 270 degrees
- moved J_FTM->R_COD_1 118.8 mm to (170.2, 108.0), turned to 90 degrees
- moved CONN->SERV_BAR1 115.5 mm to (182.9, 108.0)
- moved CONN->X-BEE1 100.3 mm to (129.5, 110.5), turned to 90 degrees
- moved CONN->DISP1 99.9 mm to (114.3, 92.7), turned to 270 degrees
- moved J_FTM->R_COD_2 98.8 mm to (121.9, 123.2), turned to 270 degrees
- moved R2 94.9 mm to (168.9, 86.4)
- moved CONN_COL1 94.3 mm to (129.5, 119.4)
- moved R1 93.4 mm to (168.9, 81.3)
- moved CONN_TIR1 91.9 mm to (113.0, 113.0), turned to 270 degrees
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Routing:
- net +5V: track 0.00 -> 267.6 mm, vias 0 -> 2
- net GND: track 0.00 -> 267.2 mm, vias 0 -> 1
- net I2C_SCLO: track 0.00 -> 53.7 mm, vias 0 -> 2
- net I2C_SDAO: track 0.00 -> 47.4 mm, vias 0 -> 1
- net TIR_GPIO: track 0.00 -> 32.8 mm
- net PAV_SERV: track 0.00 -> 32.4 mm
- net MOT_1_PWM: track 0.00 -> 32.3 mm
- net GPIO_DISPLAY_2: track 0.00 -> 30.5 mm
- net GPIO_DISPLAY_1: track 0.00 -> 30.5 mm
- net MOT_1_DIR: track 0.00 -> 30.3 mm
- net BAR_SERV: track 0.00 -> 27.1 mm
- net R_COD_2_phB: track 0.00 -> 22.9 mm
- net R_COD_2_phA: track 0.00 -> 22.9 mm
- net COL_GPIO: track 0.00 -> 21.5 mm
- net LID_TX: track 0.00 -> 19.9 mm
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
Commit message: Carte Teensy V2.0
Parts:
- added J1: Conn_01x04_Male, Connector_JST:JST_XH_B4B-XH-A_1x04_P2.50mm_Vertical, F.Cu at (189.2, 106.7)
- added J2: Conn_01x04_Male, Connector_JST:JST_XH_B4B-XH-A_1x04_P2.50mm_Vertical, F.Cu at (189.2, 97.8)
- moved CONN->MD10_MOT_1 58.0 mm to (135.9, 151.1), turned to 0 degrees
- moved U12->5 51.7 mm to (177.8, 81.3)
- moved CONN->SERV_BAR1 35.9 mm to (188.0, 143.5), turned to 270 degrees
- moved J_FTM->R_COD_1 34.9 mm to (189.2, 137.2), turned to 180 degrees
- moved J_I2C->MULTIPLEX1 34.3 mm to (189.2, 116.8)
- moved CONN->SERV_PAV1 34.3 mm to (188.0, 147.3), turned to 270 degrees
- moved ALIM_1 34.1 mm to (137.2, 81.3)
- moved J_I2C->MULTIPLEX2 31.8 mm to (189.2, 127.0)
- moved CONN->MOT_LID1 30.5 mm to (138.4, 102.9)
- moved Q1 29.6 mm to (147.3, 101.6), turned to 270 degrees
- moved CONN_TIR1 29.0 mm to (138.4, 127.0), turned to 180 degrees
- moved CONN->MD10_MOT_2 28.4 mm to (188.0, 153.7), turned to 180 degrees
- moved CONN->DISP1 25.2 mm to (133.3, 109.2), turned to 0 degrees
- moved R_Pull_D_MOT_LID1 23.1 mm to (148.2, 97.8), turned to 180 degrees
- moved J_FTM->R_COD_2 22.9 mm to (134.6, 142.2), turned to 0 degrees
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Connections:
- CARTE_MICR_COTROL1 pad 47: Net-(CARTE_MICR_COTROL1-Pad47) -> MOT_1_COD_phB
- CARTE_MICR_COTROL1 pad 48: Net-(CARTE_MICR_COTROL1-Pad48) -> MOT_1_COD_phA
- CARTE_MICR_COTROL1 pad 49: Net-(CARTE_MICR_COTROL1-Pad49) -> MOT_2_COD_phB
- CARTE_MICR_COTROL1 pad 50: Net-(CARTE_MICR_COTROL1-Pad50) -> MOT_2_COD_phA
- CONN->MD10_MOT_1 pad 1: +5V -> GND
- CONN->MD10_MOT_2 pad 1: +5V -> GND
Routing:
- net +5V: track 267.6 -> 163.8 mm, vias 2 -> 0
- net GND: track 267.2 -> 233.3 mm, vias 1 -> 4
- net I2C_SDAO: track 47.4 -> 23.6 mm, vias 1 -> 0
- net R_COD_1_phB: track 10.2 -> 32.8 mm, vias 0 -> 3
- net R_COD_1_phA: track 10.2 -> 32.6 mm
- net +12V: track 19.1 -> 40.6 mm
- net LID_TX: track 19.9 -> 0.00 mm
- net MOT_2_COD_phA: track 0.00 -> 18.6 mm
- net MOT_1_COD_phA: track 0.00 -> 17.1 mm
- net I2C_SCLO: track 53.7 -> 36.8 mm, vias 2 -> 0
- net TIR_GPIO: track 32.8 -> 16.3 mm
- net GPIO_DISPLAY_2: track 30.5 -> 14.9 mm
- net PAV_SERV: track 32.4 -> 17.1 mm
- net MOT_2_COD_phB: track 0.00 -> 14.4 mm
- net LID_RX: track 13.4 -> 0.00 mm
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
Commit message: Teensy V2.1: Carte presque prête
Parts:
- added REF**: MountingHole_3.2mm_M3, MountingHole:MountingHole_3.2mm_M3, F.Cu at (190.0, 152.0)
- added REF**: MountingHole_3.2mm_M3, MountingHole:MountingHole_3.2mm_M3, F.Cu at (133.0, 152.0)
- added REF**: MountingHole_3.2mm_M3, MountingHole:MountingHole_3.2mm_M3, F.Cu at (133.0, 81.0)
- added REF**: MountingHole_3.2mm_M3, MountingHole:MountingHole_3.2mm_M3, F.Cu at (190.0, 81.0)
- moved ALIM_1 14.0 mm to (151.1, 82.5), turned to 180 degrees
- moved CONN->MD10_MOT_2 7.73 mm to (180.3, 152.4)
- moved CONN->MD10_MOT_1 6.43 mm to (142.3, 151.1)
- moved CONN->SERV_BAR1 4.58 mm to (185.4, 139.7)
- moved J_FTM->R_COD_1 3.81 mm to (189.2, 133.3)
- moved CONN->SERV_PAV1 3.59 mm to (185.4, 144.8)
- moved J_I2C->MULTIPLEX2 2.54 mm to (189.2, 124.5)
- moved J_I2C->MULTIPLEX1 1.27 mm to (189.2, 115.6)
Routing:
- net I2C_SDAO: track 23.6 -> 39.9 mm
- net LID_TX: track 0.00 -> 16.2 mm
- net +12V: track 40.6 -> 27.2 mm
- net LID_RX: track 0.00 -> 11.5 mm
- net MOT_2_PWM: track 21.0 -> 12.1 mm
- net MOT_2_DIR: track 16.7 -> 8.53 mm
- net R_COD_1_phA: track 32.6 -> 27.3 mm, vias 0 -> 1
- net MOT_1_DIR: track 28.6 -> 24.2 mm
- net BAR_SERV: track 16.6 -> 12.5 mm
- net R_COD_1_phB: track 32.8 -> 28.9 mm, vias 3 -> 0
- net MOT_1_PWM: track 35.5 -> 31.7 mm
- net +5V: track 163.8 -> 167.5 mm
- net PAV_SERV: track 17.1 -> 13.5 mm
- net I2C_SCLO: track 36.8 -> 33.5 mm
- net GND: track 233.3 -> 235.4 mm, vias 4 -> 2
- added copper zone on B.Cu, net GND
Other:
- board outline added: 65 x 79 mm
- board text added: "+12V"
- board text added: "COD1"
- board text added: "COD2"
- board text added: "Couleur"
- board text added: "Display"
- board text added: "GND"
- board text added: "I2C"
- board text added: "LidM"
- board text added: "Lidar"
- board text added: "MC1"
- board text added: "MC2"
- board text added: "Mot1"
- board text added: "Mot2"
- board text added: "RobotA 2021 Teensy"
- board text added: "SRV1"
- board text added: "SRV2"
- board text added: "Tirette"
- board text added: "USB"
- board text added: "Victor@ENAC"
- board text added: "XBee"

Commit message: Carte Tennsy version finale
Parts:
- moved CONN->X-BEE1 1.27 mm to (133.3, 118.1)
Routing:
- net X-BEE_TX: track 17.4 -> 19.0 mm
- net R_COD_1_phA: track 27.3 -> 28.4 mm
- net LID_TX: track 16.2 -> 15.1 mm
- net GND: track 235.4 -> 236.2 mm, vias 2 -> 1
- net X-BEE_RX: track 13.9 -> 13.3 mm
Other:
- board text added: "RobotB 2021 Teensy"
- board text removed: "RobotA 2021 Teensy"
