File: kicad_robot/kicad_robot_servos_ev_pompes.kicad_pcb (KiCad board)
At the start: 2 copper layers, 99 x 61 mm, 66 parts, among them J1 Conn_I2C, J10 Conn_SERVO_3, J11 Conn_SERVO_4, J12 Conn_SERVO_5, J13 Conn_EV_1, J14 Conn_EV_2, J15 Conn_EV_3, J16 Conn_EV_4, J17 Conn_EV_5, J2 Screw_Terminal_POWER, J3 Conn_POMPE_1, J4 Conn_POMPE_5, J5 Conn_POMPE_2, J6 Conn_POMPE_3, J7 Conn_POMPE_4, J8 Conn_SERVO_1, J9 Conn_SERVO_2, Q1 IRLML0030, Q10 IRLML0030, Q2 IRLML0030, Q3 IRLML0030, Q4 IRLML0030, Q5 IRLML0030, Q6 IRLML0030, Q7 IRLML0030, Q8 IRLML0030, Q9 IRLML0030, U1 TSR_1-2450, U2 LM3940, U3 ADC128D818, U4 PCA9685PW, U5 ACS722xLCTR-05AB, U6 ACS722xLCTR-05AB, U7 ACS722xLCTR-05AB, U8 ACS722xLCTR-05AB, U9 ACS722xLCTR-05AB

Commit message: Cache de labels inutiles
Other:
- board text added: "I2C ADDR"
- board text removed: "Choix d'adresse I2C Connecter 1 Résistance / 2"

Commit message: Génération Gerber Carte Servos
Routing:
- net GND: track 496.3 -> 499.5 mm
- net /ADC_5: track 38.4 -> 39.2 mm
- net /ADC_4: track 24.0 -> 24.6 mm
- added copper zone on B.Cu, net GND
Other:
- board text added: "ENAC Robotique Robot 2021 B PCB by Rémy Brévart"
